Commit message: Add support for Spot, the Spirit and A1 examples now do not work

File: quad_simulator/spot_description/urdf/spot.urdf (robot description, URDF)
Before this commit: robot spot, 19 links, 18 joints
Links:
- link toe0: mass 0.06 -> 0.01; geometry collision sphere radius=0.037
- link toe1: mass 0.06 -> 0.01; geometry collision sphere radius=0.037
- link toe2: mass 0.06 -> 0.01; geometry collision sphere radius=0.037
- link toe3: mass 0.06 -> 0.01; geometry collision sphere radius=0.037
